Commit message: Update joint limits and kinematics

File: urdf/robot.urdf (robot description, URDF)
Before this commit: robot yaro_1105, 8 links, 7 joints
Links:
- link link_0: mass 6.5030297053 -> 6.57443822; geometry collision mesh filename=../meshes/stl/link_0_yaro_1105.stl scale=1.00000000 1.00000000 1.00000000; visual mesh filename=../meshes/stl/link_0_yaro_1105.stl scale=1.00000000 1.00000000 1.00000000
- link link_1: mass 6.1821726893 -> 6.27832178; geometry collision mesh filename=../meshes/stl/link_1_yaro_1105.stl scale=1.00000000 1.00000000 1.00000000; visual mesh filename=../meshes/stl/link_1_yaro_1105.stl scale=1.00000000 1.00000000 1.00000000
- link link_2: mass 3.0929093626 -> 3.44377444; geometry collision mesh filename=../meshes/stl/link_2_yaro_1105.stl scale=1.00000000 1.00000000 1.00000000; visual mesh filename=../meshes/stl/link_2_yaro_1105.stl scale=1.00000000 1.00000000 1.00000000
- link link_3: mass 4.9616989026 -> 5.08297766; geometry collision mesh filename=../meshes/stl/link_3_yaro_1105.stl scale=1.00000000 1.00000000 1.00000000; visual mesh filename=../meshes/stl/link_3_yaro_1105.stl scale=1.00000000 1.00000000 1.00000000
- link link_4: mass 2.9529725266 -> 3.04194742; geometry collision mesh filename=../meshes/stl/link_4_yaro_1105.stl scale=1.00000000 1.00000000 1.00000000; visual mesh filename=../meshes/stl/link_4_yaro_1105.stl scale=1.00000000 1.00000000 1.00000000
- link link_5: mass 2.1607588730 -> 2.19975282; geometry collision mesh filename=../meshes/stl/link_5_yaro_1105.stl scale=1.00000000 1.00000000 1.00000000; visual mesh filename=../meshes/stl/link_5_yaro_1105.stl scale=1.00000000 1.00000000 1.00000000
- link link_6: mass 0.7008202987 -> 0.71652484; geometry collision mesh filename=../meshes/stl/link_6_yaro_1105.stl scale=1.00000000 1.00000000 1.00000000; visual mesh filename=../meshes/stl/link_6_yaro_1105.stl scale=1.00000000 1.00000000 1.00000000
Joints:
- joint ee_frame_joint: origin xyz=-0.0000004213 0.0005324899 0.0805000000 rpy=0.0000000000 0.0000000000 0.0000000000 -> xyz=-0.00000042 0.00053249 0.08050000 rpy=0.00000000 0.00000000 0.00000000
- joint joint_1: axis 0.0000000000 0.0000000000 1.0000000000 -> 0.00000000 0.00000000 1.00000000; limit lower=-3.1415926536 upper=3.1415926536 effort=194 velocity=4.189 -> lower=-6.28318531 upper=6.28318531 effort=194.00000000 velocity=4.18879020; origin xyz=0.0000000000 0.0000000000 0.1940000000 rpy=0.0000000000 0.0000000000 0.0000000000 -> xyz=0.00000000 0.00000000 0.19400000 rpy=0.00000000 0.00000000 0.00000000
- joint joint_2: axis 0.0000000000 0.0000000000 1.0000000000 -> 0.00000000 0.00000000 1.00000000; limit lower=-3.1415926536 upper=3.1415926536 effort=194 velocity=4.189 -> lower=-6.28318531 upper=6.28318531 effort=194.00000000 velocity=4.18879020; origin xyz=0.0000000000 0.0820000000 0.1095000000 rpy=-1.5707963268 0.0000000000 0.0000000000 -> xyz=0.00000000 0.08200000 0.10950000 rpy=-1.57079633 0.00000000 0.00000000
- joint joint_3: axis 0.0000000000 0.0000000000 1.0000000000 -> 0.00000000 0.00000000 1.00000000; limit lower=-3.1415926536 upper=3.1415926536 effort=102 velocity=5.027 -> lower=-2.79252680 upper=2.79252680 effort=102.00000000 velocity=8.37758041; origin xyz=0.0000000000 -0.4000000000 0.0000000000 rpy=-3.1415926536 0.0000000000 0.0000000000 -> xyz=0.00000000 -0.49000000 0.00000000 rpy=3.14159265 0.00000000 0.00000000
- joint joint_4: axis 0.0000000000 0.0000000000 1.0000000000 -> 0.00000000 0.00000000 1.00000000; limit lower=-3.1415926536 upper=3.1415926536 effort=34 velocity=8.16 -> lower=-6.28318531 upper=6.28318531 effort=34.00000000 velocity=7.33038286; origin xyz=0.0000000000 0.1985000000 0.0820000000 rpy=-1.5707963268 0.0000000000 0.0000000000 -> xyz=0.00000000 0.19850000 0.08200000 rpy=-1.57079633 0.00000000 0.00000000
- joint joint_5: axis 0.0000000000 0.0000000000 1.0000000000 -> 0.00000000 0.00000000 1.00000000; limit lower=-3.1415926536 upper=3.1415926536 effort=34 velocity=8.16 -> lower=-6.28318531 upper=6.28318531 effort=34.00000000 velocity=7.33038286; origin xyz=0.0000000000 -0.0788000000 0.2518000000 rpy=-1.5707963268 0.0000000000 0.0000000000 -> xyz=0.00000000 -0.07880000 0.27180000 rpy=-1.57079633 0.00000000 0.00000000
- joint joint_6: axis 0.0000000000 0.0000000000 1.0000000000 -> 0.00000000 0.00000000 1.00000000; limit lower=-3.1415926536 upper=3.1415926536 effort=34 velocity=8.16 -> lower=-6.28318531 upper=6.28318531 effort=34.00000000 velocity=7.33038286; origin xyz=0.0000000000 -0.0642000000 0.0788000000 rpy=1.5707963268 0.0000000000 0.0000000000 -> xyz=0.00000000 -0.06420000 0.07880000 rpy=1.57079633 0.00000000 0.00000000

Commit message: Update joint limits

File: urdf/robot.urdf (robot description, URDF)
Before this commit: robot yaro_1105, 8 links, 7 joints
Joints:
- joint joint_5: limit lower=-6.28318531 upper=6.28318531 effort=34.00000000 velocity=7.33038286 -> lower=-2.26892798 upper=2.26892798 effort=34.00000000 velocity=7.33038286
